File: zb_pt4115.brd (EAGLE design)
At the start: 76.2 x 61 mm, 57 parts, among them IC1 68uH, IC2 68uH, IC3 68uH, IC4 68uH, IC5 68uH, IC6 220uH, U1 E72-2G4M05S1F, U2 LM2596T-ADJ/NOPB

Commit message: Add files via upload
Parts:
- IC6: value 220uH -> 68uH
Changed lines of the file:
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@@
 <drawing>
 <settings>
-<setting alwaysvectorfont="yes"/>
+<setting alwaysvectorfont="no"/>
 <setting verticaltext="up"/>
 </settings>
@@
 <attribute name="PURCHASE-URL" value="https://pricing.snapeda.com/search/part/LM2596T-ADJ/NOPB/?ref=eda" x="14.351" y="9.652" size="1.778" layer="27" rot="R90" display="off"/>
 </element>
-<element name="IC6" library="MSS1038-473MLB" package="INDPM102100X400N" value="220uH" x="26.289" y="12.827" smashed="yes">
+<element name="IC6" library="MSS1038-473MLB" package="INDPM102100X400N" value="68uH" x="26.289" y="12.827" smashed="yes">
 <attribute name="ARROW_PART_NUMBER" value="" x="26.289" y="12.827" size="1.778" layer="27" display="off"/>
 <attribute name="ARROW_PRICE-STOCK" value="" x="26.289" y="12.827" size="1.778" layer="27" display="off"/>
