File: zb_pt4115.brd (EAGLE design)
At the start: 76.2 x 61 mm, 57 parts, among them IC1 68uH, IC2 68uH, IC3 68uH, IC4 68uH, IC5 68uH, IC6 68uH, U1 E72-2G4M05S1F, U2 LM2596T-ADJ/NOPB

Commit message: Add files via upload
Parts:
- removed JTAG: CORTEX_DEBUG_SMD, SparkFun-Connectors:SAMTECH_FTSH-105-01
- removed S1: (no value), SparkFun-Switches:TACTILE_SWITCH_SMD_4.6X2.8MM
- added BTN1, BTN2, RST: MOMENTARY-SWITCH-SPST-SMD-5.2-REDUNDANT, SparkFun-Switches:TACTILE_SWITCH_SMD_5.2MM
- added C11, C12, C13, C14, C15: 100nF, SparkFun-Capacitors:0402
- added J7: (no value), SparkFun-SEWPAD16:2X4
- moved D7 25.3 mm to (67.3, 27.3), turned to 0 degrees
- moved R14 23.1 mm to (64.0, 27.3)
Connections:
- net +3V3: now also J7.1; no longer JTAG.1
- net 13: now also BTN1.3, BTN1.4
- net 14: now also BTN2.3, BTN2.4; no longer S1.3, S1.4
- net 2: now also J7.5
- net 3: now also J7.7
- net GND: now also BTN1.1, BTN1.2, BTN2.1, BTN2.2, C11.1, C12.1, C13.1, C14.1, C15.1, J7.3, RST.3, RST.4; no longer JTAG.3, JTAG.5, S1.1, S1.2
- net N$11: now also C14.2
- net N$12: now also C15.2
- net N$2: now also C11.2
- net N$7: now also C12.2
- net N$8: now also C13.2
- net RST: now also RST.1, RST.2
- net TCK: now also J7.4; no longer JTAG.4
- net TDI: now also J7.8; no longer JTAG.8
- net TDO: now also J7.6; no longer JTAG.6
- net TMS: now also J7.2; no longer JTAG.2
Routing:
- net GND: track 12.4 -> 42.1 mm, vias 86 -> 108
- net 13: track 0.00 -> 27.4 mm, vias 0 -> 2
- net TMS: track 5.01 -> 30.1 mm, vias 0 -> 1
- net 3: track 0.00 -> 24.1 mm
- net RST: track 3.93 -> 26.3 mm
- net TDI: track 9.00 -> 30.5 mm, vias 0 -> 1
- net TCK: track 7.48 -> 27.5 mm, vias 0 -> 1
- net TDO: track 8.28 -> 28.1 mm, vias 0 -> 1
- net 7: track 24.9 -> 6.75 mm, vias 2 -> 0
- net 14: track 19.3 -> 36.0 mm, vias 0 -> 2
- net 2: track 0.00 -> 7.49 mm
- net N$12: track 17.7 -> 20.4 mm
- net N$8: track 17.5 -> 20.1 mm
- net N$7: track 17.2 -> 19.7 mm
- net N$11: track 19.2 -> 21.7 mm
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
Commit message: Add files via upload
Parts:
- C11, C12, C13, C14, C15: device SparkFun-Capacitors:0402 -> SparkFun-Capacitors:0603
- MGT1, MGT2, MGT3, MGT4: value BEAGLEBONEBLACK_MOUNTING_HOLE -> MOUNT-HOLE3.0; device BeagleBone_Black_Wireless:BEAGLEBONEBLACK_MOUNTING_HOLE -> holes:3,0
- moved C11 3.69 mm to (5.84, 42.4), turned to 0 degrees
- moved C8 1.53 mm to (4.70, 12.4), turned to 180 degrees
- moved MGT1 1.53 mm to (4.32, 4.19)
- moved MGT2 1.45 mm to (72.0, 3.94)
- moved MGT4 1.20 mm to (72.0, 56.8)
- moved MGT3 0.97 mm to (4.19, 56.8)
- moved C13 0.25 mm to (19.8, 42.3)
Routing:
- net N$2: track 23.0 -> 27.5 mm
- net GND: track 42.1 -> 45.7 mm

Commit message: Add files via upload
Parts:
- moved MGT2 2.54 mm to (69.5, 4.06)
- moved MGT4 2.54 mm to (69.5, 56.6)
Routing:
- net N$3: track 31.5 -> 32.3 mm
Other:
- board size 76.2 x 61 mm -> 73.7 x 61 mm

Commit message: Add files via upload
Parts:
- R12: value (none) -> 1.5k
- R13: value (none) -> 1k
- moved MGT2 0.13 mm to (69.3, 4.06)
Routing:
- net GND: vias 108 -> 111
Other:
- board size 73.7 x 61 mm -> 74 x 61 mm
- board text added: "1. 3V3"
- board text added: "2. TMS"
- board text added: "3. GND"
- board text added: "4. TCK"
- board text added: "5. RX"
- board text added: "6. TDO"
- board text added: "7. TX"
- board text added: "8. TDI"
- board text added: "STATUS"
Changed lines of the file:
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@@
 <board>
 <plain>
-<wire x1="0" y1="0" x2="73.66" y2="0" width="0.15" layer="20"/>
-<wire x1="73.66" y1="0" x2="73.66" y2="8.128" width="0.15" layer="20"/>
-<wire x1="73.66" y1="8.128" x2="67.31" y2="8.128" width="0.15" layer="20"/>
-<wire x1="67.31" y1="8.128" x2="67.31" y2="24.511" width="0.15" layer="20"/>
-<wire x1="67.31" y1="24.511" x2="73.66" y2="24.511" width="0.15" layer="20"/>
-<wire x1="73.66" y1="24.511" x2="73.66" y2="60.96" width="0.15" layer="20"/>
-<wire x1="73.66" y1="60.96" x2="0" y2="60.96" width="0.15" layer="20"/>
-<wire x1="0" y1="60.96" x2="0" y2="0" width="0.15" layer="20"/>
 <text x="49.53" y="9.652" size="0.8128" layer="25">JLCJLCJLCJLC</text>
 <text x="12.954" y="2.794" size="1.4224" layer="25" distance="59">t.me/deaxx</text>
@@
 <text x="42.799" y="52.451" size="1.4224" layer="25" distance="59">+</text>
 <text x="48.895" y="52.451" size="1.4224" layer="25" distance="59">+</text>
-<dimension x1="73.66" y1="60.96" x2="73.66" y2="0" x3="83.566" y3="30.48" textsize="1.778" layer="1"/>
-<dimension x1="0" y1="60.96" x2="73.66" y2="60.96" x3="36.83" y3="66.04" textsize="1.778" layer="1"/>
+<text x="69.088" y="26.924" size="0.8128" layer="25" distance="36">STATUS</text>
+<text x="54.737" y="6.604" size="0.8128" layer="26" distance="36" rot="MR90">1. 3V3</text>
+<text x="54.864" y="10.668" size="0.8128" layer="26" distance="36" rot="MR90">2. TMS</text>
+<text x="57.277" y="6.604" size="0.8128" layer="26" distance="36" rot="MR90">3. GND</text>
+<text x="59.69" y="6.604" size="0.8128" layer="26" distance="36" rot="MR90">5. RX</text>
+<text x="62.23" y="6.604" size="0.8128" layer="26" distance="36" rot="MR90">7. TX</text>
+<text x="57.277" y="10.668" size="0.8128" layer="26" distance="36" rot="MR90">4. TCK</text>
+<text x="59.817" y="10.668" size="0.8128" layer="26" distance="36" rot="MR90">6. TDO</text>
+<text x="62.484" y="10.668" size="0.8128" layer="26" distance="36" rot="MR90">8. TDI</text>
+<wire x1="0" y1="55.88" x2="5.08" y2="60.96" width="0.1524" layer="20" curve="-106.260205"/>
+<wire x1="5.08" y1="60.96" x2="69.85" y2="60.96" width="0.1524" layer="20"/>
+<wire x1="69.85" y1="60.96" x2="73.914" y2="55.88" width="0.1524" layer="20" curve="-90"/>
+<wire x1="73.914" y1="55.88" x2="73.914" y2="24.511" width="0.1524" layer="20"/>
+<wire x1="73.914" y1="24.511" x2="67.818" y2="24.511" width="0.1524" layer="20"/>
+<wire x1="67.818" y1="24.511" x2="67.818" y2="8.255" width="0.1524" layer="20"/>
+<wire x1="67.818" y1="8.255" x2="73.914" y2="8.255" width="0.1524" layer="20"/>
+<wire x1="5.08" y1="0" x2="3.81" y2="0" width="0.1524" layer="20"/>
+<wire x1="5.08" y1="0" x2="0" y2="5.08" width="0.1524" layer="20" curve="-106.260205"/>
+<wire x1="0" y1="55.88" x2="0" y2="5.08" width="0.1524" layer="20"/>
+<wire x1="5.08" y1="0" x2="69.342" y2="0" width="0.1524" layer="20"/>
+<wire x1="69.342" y1="0" x2="69.723" y2="0" width="0.1524" layer="20"/>
+<wire x1="73.914" y1="8.255" x2="73.914" y2="4.318" width="0.1524" layer="20"/>
+<wire x1="73.914" y1="4.318" x2="73.914" y2="4.064" width="0.1524" layer="20"/>
+<wire x1="73.914" y1="4.318" x2="69.342" y2="0" width="0.1524" layer="20" curve="-91.659237"/>
 </plain>
 <attributes>
@@
 <attribute name="PROD_ID" value="CAP-12547" x="4.699" y="12.446" size="1.778" layer="27" rot="R180" display="off"/>
 </element>
-<element name="R12" library="adafruit" library_urn="urn:adsk.eagle:library:420" package="R0805" package3d_urn="urn:adsk.eagle:package:6240566/1" value="" x="34.163" y="18.288" smashed="yes" rot="R270">
+<element name="R12" library="adafruit" library_urn="urn:adsk.eagle:library:420" package="R0805" package3d_urn="urn:adsk.eagle:package:6240566/1" value="1.5k" x="34.163" y="18.288" smashed="yes" rot="R270">
 <attribute name="NAME" x="34.544" y="20.32" size="1.016" layer="25" rot="R90"/>
 <attribute name="VALUE" x="31.877" y="19.05" size="1.27" layer="27" rot="R270"/>
 </element>
-<element name="R13" library="adafruit" library_urn="urn:adsk.eagle:library:420" package="R0805" package3d_urn="urn:adsk.eagle:package:6240566/1" value="" x="37.719" y="18.288" smashed="yes" rot="R90">
+<element name="R13" library="adafruit" library_urn="urn:adsk.eagle:library:420" package="R0805" package3d_urn="urn:adsk.eagle:package:6240566/1" value="1k" x="37.719" y="18.288" smashed="yes" rot="R90">
 <attribute name="NAME" x="38.1" y="20.193" size="1.016" layer="25" rot="R90"/>
 <attribute name="VALUE" x="40.005" y="17.526" size="1.27" layer="27" rot="R90"/>
@@
 </element>
 <element name="R14" library="SparkFun-Resistors" library_urn="urn:adsk.eagle:library:532" package="0603" package3d_urn="urn:adsk.eagle:package:39650/1" value="2.2k" x="64.008" y="27.305" smashed="yes" rot="R180">
-<attribute name="NAME" x="64.135" y="26.543" size="1.016" layer="25" font="vector" ratio="20" rot="R180" align="bottom-center"/>
+<attribute name="NAME" x="64.135" y="29.083" size="1.016" layer="25" font="vector" ratio="20" rot="R180" align="bottom-center"/>
 <attribute name="PROD_ID" value="RES-08272" x="64.008" y="27.305" size="1.778" layer="27" rot="R180" display="off"/>
 </element>
@@
 <attribute name="POPULARITY" value="3" x="4.318" y="4.191" size="1.778" layer="27" display="off"/>
 </element>
-<element name="MGT2" library="holes" library_urn="urn:adsk.eagle:library:237" package="3,0" package3d_urn="urn:adsk.eagle:package:14277/1" value="MOUNT-HOLE3.0" x="69.469" y="4.064" smashed="yes">
-<attribute name="POPULARITY" value="3" x="69.469" y="4.064" size="1.778" layer="27" display="off"/>
+<element name="MGT2" library="holes" library_urn="urn:adsk.eagle:library:237" package="3,0" package3d_urn="urn:adsk.eagle:package:14277/1" value="MOUNT-HOLE3.0" x="69.342" y="4.064" smashed="yes">
+<attribute name="POPULARITY" value="3" x="69.342" y="4.064" size="1.778" layer="27" display="off"/>
 </element>
 <element name="MGT3" library="holes" library_urn="urn:adsk.eagle:library:237" package="3,0" package3d_urn="urn:adsk.eagle:package:14277/1" value="MOUNT-HOLE3.0" x="4.191" y="56.769" smashed="yes">
@@
 <vertex x="37.084" y="16.002"/>
 <vertex x="37.846" y="15.24"/>
-<vertex x="39.624" y="15.24"/>
-<vertex x="39.624" y="18.161"/>
+<vertex x="40.64" y="15.24"/>
+<vertex x="40.64" y="18.161"/>
 </polygon>
 <via x="39.116" y="17.653" extent="1-16" drill="0.3"/>
@@
 <wire x1="6.692" y1="40.093" x2="6.35" y2="39.751" width="0.254" layer="16"/>
 <wire x1="6.35" y1="39.751" x2="4.953" y2="39.751" width="0.254" layer="16"/>
+<via x="40.005" y="17.653" extent="1-16" drill="0.3"/>
+<via x="40.005" y="16.637" extent="1-16" drill="0.3"/>
+<via x="40.005" y="15.621" extent="1-16" drill="0.3"/>
 </signal>
 <signal name="N$4">
@@
 <contactref element="J7" pad="2"/>
 <wire x1="47.544" y1="22.939" x2="48.562" y2="22.939" width="0.2" layer="1"/>
-<wire x1="55.372" y1="22.86" x2="56.642" y2="22.86" width="0.2" layer="1"/>
+<wire x1="55.753" y1="22.86" x2="56.642" y2="22.86" width="0.2" layer="1"/>
 <wire x1="48.562" y1="22.939" x2="49.962" y2="21.539" width="0.2" layer="1"/>
-<wire x1="49.962" y1="21.539" x2="54.051" y2="21.539" width="0.2" layer="1"/>
-<wire x1="54.051" y1="21.539" x2="55.372" y2="22.86" width="0.2" layer="1"/>
+<wire x1="49.962" y1="21.539" x2="54.432" y2="21.539" width="0.2" layer="1"/>
+<wire x1="54.432" y1="21.539" x2="55.753" y2="22.86" width="0.2" layer="1"/>
 <via x="56.642" y="22.86" extent="1-16" drill="0.3"/>
 <wire x1="54.991" y1="22.352" x2="55.499" y2="22.86" width="0.2" layer="16"/>
@@
 <contactref element="BTN1" pad="3"/>
 <contactref element="BTN1" pad="4"/>
-<wire x1="55.394" y1="24.559" x2="55.394" y2="23.517" width="0.2" layer="1"/>
-<wire x1="54.483" y1="22.606" x2="53.975" y2="22.606" width="0.2" layer="1"/>
-<wire x1="55.394" y1="23.517" x2="54.483" y2="22.606" width="0.2" layer="1"/>
+<wire x1="55.394" y1="24.559" x2="55.394" y2="23.136" width="0.2" layer="1"/>
+<wire x1="54.864" y1="22.606" x2="53.975" y2="22.606" width="0.2" layer="1"/>
+<wire x1="55.394" y1="23.136" x2="54.864" y2="22.606" width="0.2" layer="1"/>
 <via x="53.975" y="22.606" extent="1-16" drill="0.3"/>
 <wire x1="53.975" y1="22.606" x2="54.591" y2="21.99" width="0.2" layer="16"/>

Commit message: Add files via upload
Parts:
- moved F1 1.02 mm to (10.2, 25.4)
Routing:
- net N$11: track 21.8 -> 23.5 mm
- net N$2: track 27.5 -> 29.2 mm
- net GND: vias 111 -> 117
