File: zb_pt4115.brd (EAGLE design)
At the start: 74 x 61 mm, 64 parts, among them IC1 68uH, IC2 68uH, IC3 68uH, IC4 68uH, IC5 68uH, IC6 68uH, U1 E72-2G4M05S1F, U2 LM2596T-ADJ/NOPB

Commit message: Add files via upload
Parts:
- removed J6: (no value), SparkFun-Connectors:1X02_2.54_SCREWTERM
- added J9: (no value), SparkFun-SEWPAD16:SCREWTERMINAL-5MM-2
Connections:
- net GND: now also J9.1; no longer J6.P2
- net VCC: now also J9.2; no longer J6.P1
Routing:
- net VCC: track 2.97 -> 1.89 mm
- net GND: vias 117 -> 124
Changed lines of the file:
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@@
 <wire x1="73.914" y1="4.318" x2="73.914" y2="4.064" width="0.1524" layer="20"/>
 <wire x1="73.914" y1="4.318" x2="69.342" y2="0" width="0.1524" layer="20" curve="-91.659237"/>
+<text x="8.001" y="19.177" size="1.9304" layer="25" distance="59">+</text>
 </plain>
 <attributes>
@@
 <attribute name="MOUSER_PART_NUMBER" value="512-SS18" x="16.51" y="20.574" size="1.778" layer="27" rot="R180" display="off"/>
 <attribute name="MOUSER_PRICE-STOCK" value="https://www.mouser.co.uk/ProductDetail/ON-Semiconductor-Fairchild/SS18?qs=mVVXn4M53U%252B25aMJheuSLA%3D%3D" x="16.51" y="20.574" size="1.778" layer="27" rot="R180" display="off"/>
-<attribute name="NAME" x="11.811" y="20.574" size="1.016" layer="25" rot="R180" align="center"/>
+<attribute name="NAME" x="16.383" y="22.86" size="1.016" layer="25" rot="R180" align="center"/>
 </element>
 <element name="C8" library="SparkFun-Capacitors" library_urn="urn:adsk.eagle:library:510" package="PANASONIC_D" package3d_urn="urn:adsk.eagle:package:37420/1" value="100uF" x="4.699" y="12.446" smashed="yes" rot="R180">
@@
 <attribute name="NAME" x="35.433" y="20.828" size="1.016" layer="25" font="vector" ratio="20" rot="R270" align="bottom-center"/>
 <attribute name="PROD_ID" value="CAP-08749" x="35.941" y="18.415" size="1.778" layer="27" rot="R270" display="off"/>
-</element>
-<element name="J6" library="SparkFun-Connectors" library_urn="urn:adsk.eagle:library:513" package="1X02_2.54_SCREWTERM" package3d_urn="urn:adsk.eagle:package:38059/1" value="" x="3.429" y="26.67" smashed="yes" rot="R270">
-<attribute name="VALUE" x="-0.635" y="27.94" size="0.6096" layer="27" font="vector" ratio="20" rot="R270"/>
 </element>
 <element name="F1" library="adafruit" package="1812" package3d_urn="urn:adsk.eagle:package:6240348/1" value="" x="10.16" y="25.4" smashed="yes" rot="R270">
@@
 <element name="J7" library="SparkFun-SEWPAD16" package="2X4" package3d_urn="urn:adsk.eagle:package:38103/1" value="" x="58.801" y="3.048" smashed="yes">
 <attribute name="VALUE" x="53.721" y="-0.635" size="0.6096" layer="27" font="vector" ratio="20"/>
+</element>
+<element name="J9" library="SparkFun-SEWPAD16" package="SCREWTERMINAL-5MM-2" package3d_urn="urn:adsk.eagle:package:38044/1" value="" x="3.429" y="26.543" smashed="yes" rot="R270">
+<attribute name="SF_SKU" value="PRT-08432" x="3.429" y="26.543" size="1.778" layer="27" rot="R270" display="off"/>
+<attribute name="VALUE" x="4.699" y="27.813" size="0.6096" layer="27" font="vector" ratio="20" rot="R270"/>
 </element>
 </elements>
@@
 <via x="2.286" y="12.446" extent="1-16" drill="0.85"/>
 <contactref element="F1" pad="1"/>
-<contactref element="F1" pad="2"/>
-<contactref element="J6" pad="P1"/>
 <polygon width="0.1524" layer="1" thermals="no">
 <vertex x="11.557" y="24.892"/>
@@
 <vertex x="15.621" y="8.509"/>
 <vertex x="15.621" y="10.668"/>
-<vertex x="3.937" y="10.668"/>
-<vertex x="3.937" y="22.225"/>
+<vertex x="4.699" y="10.668"/>
+<vertex x="4.699" y="22.225"/>
 <vertex x="11.557" y="22.225"/>
 </polygon>
@@
 <vertex x="11.557" y="29.083"/>
 </polygon>
-<wire x1="9.398" y1="30.099" x2="9.398" y2="28.208" width="0.2" layer="1"/>
-<wire x1="10.16" y1="27.446" x2="9.398" y2="28.208" width="0.2" layer="1"/>
+<wire x1="10.16" y1="29.337" x2="10.16" y2="27.446" width="0.2" layer="1"/>
+<contactref element="F1" pad="2"/>
+<contactref element="J9" pad="2"/>
 <wire x1="10.16" y1="27.446" x2="10.16" y2="23.354" width="0" layer="19" extent="1-1"/>
 </signal>
@@
 <via x="7.112" y="12.446" extent="1-16" drill="0.85" diameter="0.55"/>
 <polygon width="0.1524" layer="1" thermals="no">
-<vertex x="4.572" y="11.684"/>
+<vertex x="5.588" y="11.684"/>
 <vertex x="15.621" y="11.684"/>
 <vertex x="15.621" y="21.336"/>
-<vertex x="4.572" y="21.336"/>
+<vertex x="5.588" y="21.336"/>
 </polygon>
 <polygon width="0.1524" layer="16" thermals="no">
@@
 <vertex x="-0.635" y="-0.381"/>
 </polygon>
-<via x="5.207" y="20.701" extent="1-16" drill="0.3"/>
 <via x="6.223" y="20.701" extent="1-16" drill="0.3"/>
 <via x="7.239" y="20.701" extent="1-16" drill="0.3"/>
 <via x="8.255" y="20.701" extent="1-16" drill="0.3"/>
-<via x="9.398" y="20.701" extent="1-16" drill="0.3"/>
-<via x="10.541" y="20.701" extent="1-16" drill="0.3"/>
-<via x="5.207" y="19.558" extent="1-16" drill="0.3"/>
-<via x="5.207" y="18.415" extent="1-16" drill="0.3"/>
-<via x="5.207" y="17.272" extent="1-16" drill="0.3"/>
-<via x="5.207" y="16.129" extent="1-16" drill="0.3"/>
+<via x="9.271" y="20.701" extent="1-16" drill="0.3"/>
+<via x="10.414" y="20.701" extent="1-16" drill="0.3"/>
+<via x="11.557" y="20.701" extent="1-16" drill="0.3"/>
+<via x="6.223" y="19.558" extent="1-16" drill="0.3"/>
+<via x="6.223" y="18.415" extent="1-16" drill="0.3"/>
+<via x="6.223" y="17.272" extent="1-16" drill="0.3"/>
+<via x="6.223" y="16.129" extent="1-16" drill="0.3"/>
 <polygon width="0.1524" layer="1" thermals="no">
 <vertex x="33.02" y="10.414"/>
@@
 <via x="39.116" y="16.637" extent="1-16" drill="0.3"/>
 <via x="39.116" y="15.621" extent="1-16" drill="0.3"/>
-<via x="6.223" y="16.129" extent="1-16" drill="0.3"/>
-<via x="6.223" y="17.272" extent="1-16" drill="0.3"/>
-<via x="6.223" y="18.415" extent="1-16" drill="0.3"/>
-<via x="6.223" y="19.558" extent="1-16" drill="0.3"/>
+<via x="7.239" y="16.129" extent="1-16" drill="0.3"/>
+<via x="7.239" y="17.272" extent="1-16" drill="0.3"/>
+<via x="7.239" y="18.415" extent="1-16" drill="0.3"/>
 <via x="7.239" y="19.558" extent="1-16" drill="0.3"/>
 <via x="8.255" y="19.558" extent="1-16" drill="0.3"/>
-<via x="9.398" y="19.558" extent="1-16" drill="0.3"/>
-<via x="10.541" y="19.558" extent="1-16" drill="0.3"/>
-<via x="7.239" y="18.415" extent="1-16" drill="0.3"/>
+<via x="9.271" y="19.558" extent="1-16" drill="0.3"/>
+<via x="10.414" y="19.558" extent="1-16" drill="0.3"/>
+<via x="11.557" y="19.558" extent="1-16" drill="0.3"/>
 <via x="8.255" y="18.415" extent="1-16" drill="0.3"/>
-<via x="9.398" y="18.415" extent="1-16" drill="0.3"/>
-<via x="10.541" y="18.415" extent="1-16" drill="0.3"/>
-<via x="7.239" y="17.272" extent="1-16" drill="0.3"/>
+<via x="9.271" y="18.415" extent="1-16" drill="0.3"/>
+<via x="10.414" y="18.415" extent="1-16" drill="0.3"/>
+<via x="11.557" y="18.415" extent="1-16" drill="0.3"/>
 <via x="8.255" y="17.272" extent="1-16" drill="0.3"/>
-<via x="9.398" y="17.272" extent="1-16" drill="0.3"/>
-<via x="10.541" y="17.272" extent="1-16" drill="0.3"/>
-<via x="7.239" y="16.129" extent="1-16" drill="0.3"/>
+<via x="9.271" y="17.272" extent="1-16" drill="0.3"/>
+<via x="10.414" y="17.272" extent="1-16" drill="0.3"/>
+<via x="11.557" y="17.272" extent="1-16" drill="0.3"/>
 <via x="8.255" y="16.129" extent="1-16" drill="0.3"/>
-<via x="9.398" y="16.129" extent="1-16" drill="0.3"/>
-<via x="10.541" y="16.129" extent="1-16" drill="0.3"/>
-<contactref element="J6" pad="P2"/>
+<via x="9.271" y="16.129" extent="1-16" drill="0.3"/>
+<via x="10.414" y="16.129" extent="1-16" drill="0.3"/>
+<via x="11.557" y="16.129" extent="1-16" drill="0.3"/>
 <polygon width="0.1524" layer="16" thermals="no">
 <vertex x="18.288" y="41.275"/>
@@
 <polygon width="0.1524" layer="16" thermals="no">
 <vertex x="32.385" y="41.275"/>
-<vertex x="32.385" y="37.084"/>
-<vertex x="35.687" y="33.782"/>
+<vertex x="32.385" y="36.703"/>
+<vertex x="35.687" y="33.401"/>
 <vertex x="35.687" y="28.067"/>
 <vertex x="41.783" y="28.067"/>
@@
 <polygon width="0.1524" layer="16" thermals="no">
 <vertex x="46.482" y="41.275"/>
-<vertex x="46.482" y="37.211"/>
-<vertex x="49.911" y="33.782"/>
+<vertex x="46.482" y="36.703"/>
+<vertex x="49.911" y="33.274"/>
 <vertex x="49.911" y="28.321"/>
 <vertex x="56.007" y="28.321"/>
@@
 <vertex x="4.318" y="36.576"/>
 </polygon>
+<contactref element="J9" pad="1"/>
+<via x="41.021" y="2.667" extent="1-16" drill="0.3"/>
+<via x="62.611" y="6.477" extent="1-16" drill="0.3"/>
+<via x="4.953" y="36.576" extent="1-16" drill="0.35"/>
+<via x="18.923" y="36.703" extent="1-16" drill="0.35"/>
+<via x="32.766" y="36.703" extent="1-16" drill="0.35"/>
+<via x="46.863" y="36.83" extent="1-16" drill="0.35"/>
+<via x="61.087" y="36.83" extent="1-16" drill="0.35"/>
 </signal>
 <signal name="N$4">
