File: zb_pt4115.sch (EAGLE design)
At the start: 57 parts, among them IC1 68uH, IC2 68uH, IC3 68uH, IC4 68uH, IC5 68uH, IC6 220uH, U1 E72-2G4M05S1F, U2 LM2596T-ADJ/NOPB

Commit message: Add files via upload
Parts:
- IC6: value 220uH -> 68uH
Changed lines of the file:
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@@
 <part name="GND13" library="supply1" library_urn="urn:adsk.eagle:library:371" deviceset="GND" device=""/>
 <part name="P+6" library="supply1" library_urn="urn:adsk.eagle:library:371" deviceset="VCC" device="" value="12V"/>
-<part name="IC6" library="MSS1038-473MLB" deviceset="MSS1038-473MLB" device="" value="220uH"/>
+<part name="IC6" library="MSS1038-473MLB" deviceset="MSS1038-473MLB" device="" value="68uH"/>
 <part name="+3V1" library="supply1" library_urn="urn:adsk.eagle:library:371" deviceset="+3V3" device=""/>
 <part name="C7" library="SparkFun-Capacitors" library_urn="urn:adsk.eagle:library:510" deviceset="100UF-POLAR" device="-25V-20%(ELEC)" package3d_urn="urn:adsk.eagle:package:37420/1" value="100uF"/>

Commit message: Add files via upload
Parts:
- removed JTAG: CORTEX_DEBUG_SMD, SparkFun-Connectors:CORTEX_DEBUG_SMD
- removed S1: (no value), SparkFun-Switches:MOMENTARY-SWITCH-SPST-2-SMD-4.6X2.8MM
- added BTN1, BTN2, RST: MOMENTARY-SWITCH-SPST-SMD-5.2-REDUNDANT, SparkFun-Switches:MOMENTARY-SWITCH-SPST-SMD-5.2-REDUNDANT
- added C11, C12, C13, C14, C15: 100nF, SparkFun-Capacitors:470NF-0402-16V-10%
- added J7: (no value), SparkFun-SEWPAD16:CONN_04X2
Connections:
- net +3V3: now also J7.1; no longer JTAG.VCC
- net 13: now also BTN1.2
- net 14: now also BTN2.2; no longer S1.3, S1.4
- net 2: now also J7.5
- net 3: now also J7.7
- net GND: now also BTN1.1, BTN2.1, C11.1, C12.1, C13.1, C14.1, C15.1, J7.3, RST.2; no longer JTAG.GND@3, JTAG.GND@5, S1.1, S1.2
- net N$11: now also C14.2
- net N$12: now also C15.2
- net N$2: now also C11.2
- net N$7: now also C12.2
- net N$8: now also C13.2
- net RST: now also RST.1
- net TCK: now also J7.4; no longer JTAG.SWDCLK/TCK
- net TDI: now also J7.8; no longer JTAG.NC/TDI
- net TDO: now also J7.6; no longer JTAG.SWO/TDO
- net TMS: now also J7.2; no longer JTAG.SWDIO/TMS
Other:
- moved on the sheet: C1, C10, C2, C3, C4, C5, C6, C7, C8, C9, D7, F1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

Commit message: Add files via upload
Parts:
- C11, C12, C13, C14, C15: device SparkFun-Capacitors:470NF-0402-16V-10% -> SparkFun-Capacitors:2.2NF/2200PF-0603-50V-10%
- MGT1, MGT2, MGT3, MGT4: value BEAGLEBONEBLACK_MOUNTING_HOLE -> MOUNT-HOLE3.0; device BeagleBone_Black_Wireless:BEAGLEBONEBLACK_MOUNTING_HOLE -> holes:MOUNT-HOLE3.0
Changed lines of the file:
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@@
 <part name="GND19" library="supply1" library_urn="urn:adsk.eagle:library:371" deviceset="GND" device=""/>
 <part name="GND20" library="supply1" library_urn="urn:adsk.eagle:library:371" deviceset="GND" device=""/>
-<part name="MGT1" library="BeagleBone_Black_Wireless" library_urn="urn:adsk.eagle:library:6644236" deviceset="BEAGLEBONEBLACK_MOUNTING_HOLE" device="" package3d_urn="urn:adsk.eagle:package:6644362/2"/>
-<part name="MGT2" library="BeagleBone_Black_Wireless" library_urn="urn:adsk.eagle:library:6644236" deviceset="BEAGLEBONEBLACK_MOUNTING_HOLE" device="" package3d_urn="urn:adsk.eagle:package:6644362/2"/>
-<part name="MGT3" library="BeagleBone_Black_Wireless" library_urn="urn:adsk.eagle:library:6644236" deviceset="BEAGLEBONEBLACK_MOUNTING_HOLE" device="" package3d_urn="urn:adsk.eagle:package:6644362/2"/>
-<part name="MGT4" library="BeagleBone_Black_Wireless" library_urn="urn:adsk.eagle:library:6644236" deviceset="BEAGLEBONEBLACK_MOUNTING_HOLE" device="" package3d_urn="urn:adsk.eagle:package:6644362/2"/>
+<part name="MGT1" library="holes" library_urn="urn:adsk.eagle:library:237" deviceset="MOUNT-HOLE" device="3.0" package3d_urn="urn:adsk.eagle:package:14277/1"/>
+<part name="MGT2" library="holes" library_urn="urn:adsk.eagle:library:237" deviceset="MOUNT-HOLE" device="3.0" package3d_urn="urn:adsk.eagle:package:14277/1"/>
+<part name="MGT3" library="holes" library_urn="urn:adsk.eagle:library:237" deviceset="MOUNT-HOLE" device="3.0" package3d_urn="urn:adsk.eagle:package:14277/1" value="MOUNT-HOLE3.0"/>
+<part name="MGT4" library="holes" library_urn="urn:adsk.eagle:library:237" deviceset="MOUNT-HOLE" device="3.0" package3d_urn="urn:adsk.eagle:package:14277/1"/>
 <part name="BTN2" library="SparkFun-Switches" library_urn="urn:adsk.eagle:library:535" deviceset="MOMENTARY-SWITCH-SPST" device="-SMD-5.2-REDUNDANT" package3d_urn="urn:adsk.eagle:package:40167/1"/>
 <part name="RST" library="SparkFun-Switches" library_urn="urn:adsk.eagle:library:535" deviceset="MOMENTARY-SWITCH-SPST" device="-SMD-5.2-REDUNDANT" package3d_urn="urn:adsk.eagle:package:40167/1"/>
@@
 <part name="BTN1" library="SparkFun-Switches" library_urn="urn:adsk.eagle:library:535" deviceset="MOMENTARY-SWITCH-SPST" device="-SMD-5.2-REDUNDANT" package3d_urn="urn:adsk.eagle:package:40167/1"/>
 <part name="GND22" library="supply1" library_urn="urn:adsk.eagle:library:371" deviceset="GND" device=""/>
-<part name="C11" library="SparkFun-Capacitors" library_urn="urn:adsk.eagle:library:510" deviceset="470NF" device="-0402-16V-10%" package3d_urn="urn:adsk.eagle:package:37413/1" value="100nF"/>
-<part name="C12" library="SparkFun-Capacitors" library_urn="urn:adsk.eagle:library:510" deviceset="470NF" device="-0402-16V-10%" package3d_urn="urn:adsk.eagle:package:37413/1" value="100nF"/>
-<part name="C13" library="SparkFun-Capacitors" library_urn="urn:adsk.eagle:library:510" deviceset="470NF" device="-0402-16V-10%" package3d_urn="urn:adsk.eagle:package:37413/1" value="100nF"/>
-<part name="C14" library="SparkFun-Capacitors" library_urn="urn:adsk.eagle:library:510" deviceset="470NF" device="-0402-16V-10%" package3d_urn="urn:adsk.eagle:package:37413/1" value="100nF"/>
-<part name="C15" library="SparkFun-Capacitors" library_urn="urn:adsk.eagle:library:510" deviceset="470NF" device="-0402-16V-10%" package3d_urn="urn:adsk.eagle:package:37413/1" value="100nF"/>
+<part name="C11" library="SparkFun-Capacitors" library_urn="urn:adsk.eagle:library:510" deviceset="2.2NF/2200PF" device="-0603-50V-10%" package3d_urn="urn:adsk.eagle:package:37414/1" value="100nF"/>
+<part name="C12" library="SparkFun-Capacitors" library_urn="urn:adsk.eagle:library:510" deviceset="2.2NF/2200PF" device="-0603-50V-10%" package3d_urn="urn:adsk.eagle:package:37414/1" value="100nF"/>
+<part name="C13" library="SparkFun-Capacitors" library_urn="urn:adsk.eagle:library:510" deviceset="2.2NF/2200PF" device="-0603-50V-10%" package3d_urn="urn:adsk.eagle:package:37414/1" value="100nF"/>
+<part name="C14" library="SparkFun-Capacitors" library_urn="urn:adsk.eagle:library:510" deviceset="2.2NF/2200PF" device="-0603-50V-10%" package3d_urn="urn:adsk.eagle:package:37414/1" value="100nF"/>
+<part name="C15" library="SparkFun-Capacitors" library_urn="urn:adsk.eagle:library:510" deviceset="2.2NF/2200PF" device="-0603-50V-10%" package3d_urn="urn:adsk.eagle:package:37414/1" value="100nF"/>
 <part name="GND18" library="supply1" library_urn="urn:adsk.eagle:library:371" deviceset="GND" device=""/>
 <part name="GND23" library="supply1" library_urn="urn:adsk.eagle:library:371" deviceset="GND" device=""/>

Commit message: Add files via upload
Parts:
- R12: value (none) -> 1.5k
- R13: value (none) -> 1k
Changed lines of the file:
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@@
 <part name="+3V3" library="supply1" library_urn="urn:adsk.eagle:library:371" deviceset="+3V3" device=""/>
 <part name="GND15" library="supply1" library_urn="urn:adsk.eagle:library:371" deviceset="GND" device=""/>
-<part name="R12" library="adafruit" library_urn="urn:adsk.eagle:library:420" deviceset="R-US_" device="R0805" package3d_urn="urn:adsk.eagle:package:6240566/1"/>
-<part name="R13" library="adafruit" library_urn="urn:adsk.eagle:library:420" deviceset="R-US_" device="R0805" package3d_urn="urn:adsk.eagle:package:6240566/1"/>
+<part name="R12" library="adafruit" library_urn="urn:adsk.eagle:library:420" deviceset="R-US_" device="R0805" package3d_urn="urn:adsk.eagle:package:6240566/1" value="1.5k"/>
+<part name="R13" library="adafruit" library_urn="urn:adsk.eagle:library:420" deviceset="R-US_" device="R0805" package3d_urn="urn:adsk.eagle:package:6240566/1" value="1k"/>
 <part name="GND16" library="supply1" library_urn="urn:adsk.eagle:library:371" deviceset="GND" device=""/>
 <part name="C9" library="SparkFun-Capacitors" library_urn="urn:adsk.eagle:library:510" deviceset="560PF" device="-0603-50V-5%" package3d_urn="urn:adsk.eagle:package:37414/1" value="560pF"/>

Commit message: Add files via upload
Parts:
- removed J6: (no value), SparkFun-Connectors:CONN_022.54MM_SCREWTERM
- added J9: (no value), SparkFun-SEWPAD16:CONN_025MM
Connections:
- net GND: now also J9.1; no longer J6.2
- net VCC: now also J9.2; no longer J6.1
Other:
- moved on the sheet: F1
Changed lines of the file:
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@@
 <part name="GND16" library="supply1" library_urn="urn:adsk.eagle:library:371" deviceset="GND" device=""/>
 <part name="C9" library="SparkFun-Capacitors" library_urn="urn:adsk.eagle:library:510" deviceset="560PF" device="-0603-50V-5%" package3d_urn="urn:adsk.eagle:package:37414/1" value="560pF"/>
-<part name="J6" library="SparkFun-Connectors" library_urn="urn:adsk.eagle:library:513" deviceset="CONN_02" device="2.54MM_SCREWTERM" package3d_urn="urn:adsk.eagle:package:38059/1"/>
 <part name="GND17" library="supply1" library_urn="urn:adsk.eagle:library:371" deviceset="GND" device=""/>
 <part name="F1" library="adafruit" deviceset="PTCFUSE" device="-1812" package3d_urn="urn:adsk.eagle:package:6240348/1"/>
@@
 <part name="GND27" library="supply1" library_urn="urn:adsk.eagle:library:371" deviceset="GND" device=""/>
 <part name="+3V4" library="supply1" library_urn="urn:adsk.eagle:library:371" deviceset="+3V3" device=""/>
+<part name="J9" library="SparkFun-SEWPAD16" deviceset="CONN_02" device="5MM" package3d_urn="urn:adsk.eagle:package:38044/1"/>
 </parts>
 <sheets>
@@
 <attribute name="VALUE" x="58.039" y="143.764" size="1.778" layer="96" font="vector" rot="R90"/>
 </instance>
-<instance part="J6" gate="G$1" x="22.86" y="106.68" smashed="yes" rot="R270">
-<attribute name="VALUE" x="18.034" y="109.22" size="1.778" layer="96" font="vector" rot="R270"/>
-<attribute name="NAME" x="28.448" y="109.22" size="1.778" layer="95" font="vector" rot="R270"/>
-</instance>
-<instance part="GND17" gate="1" x="30.48" y="91.44" smashed="yes">
-<attribute name="VALUE" x="27.94" y="88.9" size="1.778" layer="96"/>
-</instance>
-<instance part="F1" gate="G$1" x="17.78" y="91.44" smashed="yes">
-<attribute name="VALUE" x="13.97" y="90.17" size="1.778" layer="96"/>
-<attribute name="NAME" x="13.97" y="96.52" size="1.778" layer="95"/>
-</instance>
-<instance part="P+7" gate="VCC" x="7.62" y="93.98" smashed="yes" rot="R90">
-<attribute name="VALUE" x="10.16" y="91.44" size="1.778" layer="96" rot="R180"/>
+<instance part="GND17" gate="1" x="35.56" y="104.14" smashed="yes">
+<attribute name="VALUE" x="33.02" y="101.6" size="1.778" layer="96"/>
+</instance>
+<instance part="F1" gate="G$1" x="22.86" y="104.14" smashed="yes">
+<attribute name="VALUE" x="19.05" y="102.87" size="1.778" layer="96"/>
+<attribute name="NAME" x="19.05" y="109.22" size="1.778" layer="95"/>
+</instance>
+<instance part="P+7" gate="VCC" x="12.7" y="106.68" smashed="yes" rot="R90">
+<attribute name="VALUE" x="15.24" y="104.14" size="1.778" layer="96" rot="R180"/>
 </instance>
 <instance part="C10" gate="G$1" x="111.76" y="116.84" smashed="yes">
@@
 <instance part="+3V4" gate="G$1" x="144.78" y="60.96" smashed="yes">
 <attribute name="VALUE" x="147.32" y="55.88" size="1.778" layer="96" rot="R90"/>
+</instance>
+<instance part="J9" gate="G$1" x="30.48" y="96.52" smashed="yes" rot="R90">
+<attribute name="VALUE" x="35.306" y="93.98" size="1.778" layer="96" font="vector" rot="R90"/>
+<attribute name="NAME" x="24.892" y="93.98" size="1.778" layer="95" font="vector" rot="R90"/>
 </instance>
 </instances>
@@
 <segment>
 <pinref part="F1" gate="G$1" pin="1"/>
-<wire x1="12.7" y1="93.98" x2="10.16" y2="93.98" width="0.1524" layer="91"/>
+<wire x1="17.78" y1="106.68" x2="15.24" y2="106.68" width="0.1524" layer="91"/>
 <pinref part="P+7" gate="VCC" pin="VCC"/>
 </segment>
 <segment>
 <pinref part="F1" gate="G$1" pin="2"/>
-<pinref part="J6" gate="G$1" pin="1"/>
-<wire x1="22.86" y1="93.98" x2="22.86" y2="99.06" width="0.1524" layer="91"/>
-<label x="22.86" y="93.98" size="1.778" layer="95" rot="R90"/>
+<pinref part="J9" gate="G$1" pin="2"/>
+<wire x1="27.94" y1="106.68" x2="27.94" y2="104.14" width="0.1524" layer="91"/>
 </segment>
 </net>
@@
 </segment>
 <segment>
-<pinref part="J6" gate="G$1" pin="2"/>
-<wire x1="25.4" y1="99.06" x2="25.4" y2="93.98" width="0.1524" layer="91"/>
-<wire x1="25.4" y1="93.98" x2="30.48" y2="93.98" width="0.1524" layer="91"/>
+<wire x1="30.48" y1="106.68" x2="35.56" y2="106.68" width="0.1524" layer="91"/>
 <pinref part="GND17" gate="1" pin="GND"/>
-</segment>
-<segment>
+<pinref part="J9" gate="G$1" pin="1"/>
+<wire x1="30.48" y1="106.68" x2="30.48" y2="104.14" width="0.1524" layer="91"/>
+</segment>
+<segment>
