File: v1.1/zb_pt4115_v1.1.brd (EAGLE design)
At the start: 74 x 61 mm, 78 parts, among them IC1 68uH, IC2 68uH, IC3 68uH, IC4 68uH, IC5 68uH, IC6 68uH, U1 E72-2G4M05S1F, U2 LM2596T-ADJ/NOPB

Commit message: Add files via upload
Routing:
- net 13: track 18.9 -> 18.4 mm
- net GND: vias 115 -> 140
Changed lines of the file:
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@@
 <via x="6.223" y="16.129" extent="1-16" drill="0.3"/>
 <polygon width="0.1524" layer="1" thermals="no">
-<vertex x="33.02" y="10.414"/>
-<vertex x="33.02" y="7.112"/>
+<vertex x="33.401" y="10.414"/>
+<vertex x="33.401" y="7.112"/>
 <vertex x="43.942" y="7.112"/>
 <vertex x="43.942" y="10.033"/>
@@
 <vertex x="9.652" y="0.254"/>
 <vertex x="9.652" y="6.477"/>
-<vertex x="33.02" y="6.477"/>
-<vertex x="33.02" y="8.255"/>
+<vertex x="33.401" y="6.477"/>
+<vertex x="33.401" y="8.255"/>
 <vertex x="41.275" y="8.255"/>
 </polygon>
@@
 <via x="61.214" y="16.383" extent="1-16" drill="0.3"/>
 <via x="57.404" y="16.383" extent="1-16" drill="0.3"/>
-<via x="61.214" y="19.431" extent="1-16" drill="0.3"/>
+<via x="52.07" y="23.241" extent="1-16" drill="0.3"/>
 <via x="53.594" y="13.335" extent="1-16" drill="0.3"/>
 <via x="49.784" y="13.335" extent="1-16" drill="0.3"/>
@@
 <via x="19.304" y="3.175" extent="1-16" drill="0.3"/>
 <via x="43.434" y="21.463" extent="1-16" drill="0.3"/>
+<via x="42.164" y="8.509" extent="1-16" drill="0.3"/>
+<via x="42.164" y="9.525" extent="1-16" drill="0.3"/>
+<via x="56.515" y="23.241" extent="1-16" drill="0.3"/>
+<via x="58.166" y="23.241" extent="1-16" drill="0.3"/>
+<via x="59.182" y="9.525" extent="1-16" drill="0.3"/>
+<via x="51.689" y="9.525" extent="1-16" drill="0.3"/>
+<via x="51.689" y="13.335" extent="1-16" drill="0.3"/>
+<via x="51.562" y="16.383" extent="1-16" drill="0.3"/>
+<via x="59.182" y="13.335" extent="1-16" drill="0.3"/>
+<via x="59.182" y="16.383" extent="1-16" drill="0.3"/>
+<via x="61.214" y="19.431" extent="1-16" drill="0.3"/>
+<via x="10.414" y="5.715" extent="1-16" drill="0.3"/>
+<via x="10.414" y="1.016" extent="1-16" drill="0.3"/>
+<via x="10.414" y="3.302" extent="1-16" drill="0.3"/>
+<via x="19.304" y="4.445" extent="1-16" drill="0.3"/>
+<via x="52.197" y="5.461" extent="1-16" drill="0.3"/>
+<via x="52.451" y="1.143" extent="1-16" drill="0.3"/>
+<via x="45.212" y="16.383" extent="1-16" drill="0.3"/>
+<via x="43.434" y="14.478" extent="1-16" drill="0.3"/>
+<via x="45.212" y="14.478" extent="1-16" drill="0.3"/>
+<via x="43.434" y="18.034" extent="1-16" drill="0.3"/>
+<via x="50.8" y="5.461" extent="1-16" drill="0.3"/>
+<via x="50.927" y="3.175" extent="1-16" drill="0.3"/>
+<via x="51.054" y="1.143" extent="1-16" drill="0.3"/>
+<via x="51.308" y="21.717" extent="1-16" drill="0.3"/>
 </signal>
 <signal name="N$4">
@@
 <wire x1="46.855" y1="19.639" x2="47.544" y2="19.639" width="0.2" layer="1"/>
 <contactref element="J7" pad="8"/>
-<wire x1="57.231" y1="18.877" x2="49.83" y2="18.877" width="0.2" layer="1"/>
-<wire x1="49.83" y1="18.877" x2="49.068" y2="19.639" width="0.2" layer="1"/>
-<wire x1="47.544" y1="19.639" x2="49.068" y2="19.639" width="0.2" layer="1"/>
+<wire x1="57.231" y1="18.877" x2="50.592" y2="18.877" width="0.2" layer="1"/>
+<wire x1="50.592" y1="18.877" x2="49.83" y2="19.639" width="0.2" layer="1"/>
+<wire x1="47.544" y1="19.639" x2="49.83" y2="19.639" width="0.2" layer="1"/>
 <wire x1="57.912" y1="19.558" x2="57.231" y2="18.877" width="0.2" layer="1"/>
 <via x="57.912" y="19.558" extent="1-16" drill="0.3"/>
@@
 <wire x1="55.791" y1="6.6236875" x2="55.791" y2="18.453" width="0.2" layer="16"/>
 <via x="56.896" y="19.558" extent="1-16" drill="0.3"/>
-<wire x1="56.68" y1="19.342" x2="49.957" y2="19.342" width="0.2" layer="1"/>
-<wire x1="49.957" y1="19.342" x2="48.56" y2="20.739" width="0.2" layer="1"/>
-<wire x1="48.56" y1="20.739" x2="47.544" y2="20.739" width="0.2" layer="1"/>
+<wire x1="56.68" y1="19.342" x2="50.719" y2="19.342" width="0.2" layer="1"/>
+<wire x1="50.719" y1="19.342" x2="49.322" y2="20.739" width="0.2" layer="1"/>
+<wire x1="49.322" y1="20.739" x2="47.544" y2="20.739" width="0.2" layer="1"/>
 <wire x1="56.896" y1="19.558" x2="56.68" y2="19.342" width="0.2" layer="1"/>
 </signal>
@@
 <wire x1="55.391" y1="19.069" x2="56.769" y2="20.447" width="0.2" layer="16"/>
 <wire x1="55.391" y1="6.458" x2="55.391" y2="19.069" width="0.2" layer="16"/>
-<wire x1="47.544" y1="21.839" x2="48.646" y2="21.839" width="0.2" layer="1"/>
-<wire x1="48.895" y1="21.59" x2="48.895" y2="20.9696875" width="0.2" layer="1"/>
-<wire x1="48.646" y1="21.839" x2="48.895" y2="21.59" width="0.2" layer="1"/>
-<wire x1="48.895" y1="20.9696875" x2="50.1226875" y2="19.742" width="0.2" layer="1"/>
-<wire x1="50.1226875" y1="19.742" x2="56.064" y2="19.742" width="0.2" layer="1"/>
+<wire x1="47.544" y1="21.839" x2="48.9" y2="21.839" width="0.2" layer="1"/>
+<wire x1="48.9" y1="21.839" x2="50.997" y2="19.742" width="0.2" layer="1"/>
+<wire x1="50.997" y1="19.742" x2="56.064" y2="19.742" width="0.2" layer="1"/>
 </signal>
 <signal name="TMS">
@@
 <contactref element="J7" pad="2"/>
 <wire x1="47.544" y1="22.939" x2="48.435" y2="22.939" width="0.2" layer="1"/>
-<wire x1="50.419" y1="20.142" x2="55.575" y2="20.142" width="0.2" layer="1"/>
+<wire x1="51.232" y1="20.142" x2="55.575" y2="20.142" width="0.2" layer="1"/>
 <wire x1="55.88" y1="20.447" x2="55.575" y2="20.142" width="0.2" layer="1"/>
 <via x="55.88" y="20.447" extent="1-16" drill="0.3"/>
@@
 <wire x1="55.88" y1="20.32" x2="54.991" y2="19.431" width="0.2" layer="16"/>
 <wire x1="54.991" y1="4.318" x2="54.991" y2="19.431" width="0.2" layer="16"/>
-<wire x1="49.295" y1="21.266" x2="50.419" y2="20.142" width="0.2" layer="1"/>
-<wire x1="48.435" y1="22.939" x2="49.295" y2="22.079" width="0.2" layer="1"/>
-<wire x1="49.295" y1="22.079" x2="49.295" y2="21.266" width="0.2" layer="1"/>
+<wire x1="48.435" y1="22.939" x2="51.232" y2="20.142" width="0.2" layer="1"/>
 </signal>
 <signal name="13">
@@
 <contactref element="BTN1" pad="4"/>
 <wire x1="55.394" y1="24.559" x2="55.394" y2="23.136" width="0.2" layer="1"/>
-<wire x1="54.229" y1="21.971" x2="55.394" y2="23.136" width="0.2" layer="1"/>
+<wire x1="54.864" y1="22.606" x2="55.394" y2="23.136" width="0.2" layer="1"/>
 <wire x1="45.466" y1="18.923" x2="45.466" y2="24.511" width="0.2" layer="1"/>
 <wire x1="45.466" y1="24.511" x2="48.26" y2="24.511" width="0.2" layer="1"/>
 <wire x1="48.768" y1="24.003" x2="48.768" y2="23.2986875" width="0.2" layer="1"/>
 <wire x1="48.26" y1="24.511" x2="48.768" y2="24.003" width="0.2" layer="1"/>
-<wire x1="48.768" y1="23.2986875" x2="50.0956875" y2="21.971" width="0.2" layer="1"/>
-<wire x1="50.0956875" y1="21.971" x2="54.229" y2="21.971" width="0.2" layer="1"/>
+<wire x1="48.768" y1="23.2986875" x2="49.4606875" y2="22.606" width="0.2" layer="1"/>
+<wire x1="49.4606875" y1="22.606" x2="54.864" y2="22.606" width="0.2" layer="1"/>
 </signal>
 <signal name="7">
@@
 <polygon width="0.1524" layer="1" thermals="no">
 <vertex x="17.272" y="12.446"/>
-<vertex x="17.272" y="7.112"/>
-<vertex x="24.003" y="7.112"/>
+<vertex x="17.272" y="7.62"/>
+<vertex x="24.003" y="7.62"/>
 <vertex x="24.003" y="21.336"/>
 <vertex x="17.526" y="21.336"/>
@@
 <contactref element="C9" pad="2"/>
 <polygon width="0.1524" layer="1" thermals="no">
-<vertex x="32.385" y="7.112"/>
-<vertex x="28.575" y="7.112"/>
+<vertex x="32.385" y="7.62"/>
+<vertex x="28.575" y="7.62"/>
 <vertex x="28.575" y="18.161"/>
 <vertex x="36.449" y="18.161"/>
@@
 <via x="38.608" y="4.699" extent="1-16" drill="0.3"/>
 <via x="44.069" y="4.572" extent="1-16" drill="0.3"/>
-<wire x1="20.701" y1="4.699" x2="26.924" y2="4.699" width="0.2" layer="1"/>
-<wire x1="26.924" y1="4.699" x2="32.893" y2="4.699" width="0.2" layer="1"/>
-<wire x1="32.893" y1="4.699" x2="38.608" y2="4.699" width="0.2" layer="1"/>
-<wire x1="38.608" y1="4.699" x2="43.942" y2="4.699" width="0.2" layer="1"/>
-<wire x1="43.942" y1="4.699" x2="44.069" y2="4.572" width="0.2" layer="1"/>
+<wire x1="26.797" y1="4.826" x2="26.924" y2="4.699" width="0.2" layer="1"/>
+<wire x1="26.797" y1="4.826" x2="20.828" y2="4.826" width="0.2" layer="1"/>
+<wire x1="20.701" y1="4.699" x2="20.828" y2="4.826" width="0.2" layer="1"/>
+<wire x1="32.766" y1="4.826" x2="27.051" y2="4.826" width="0.2" layer="1"/>
+<wire x1="26.924" y1="4.699" x2="27.051" y2="4.826" width="0.2" layer="1"/>
+<wire x1="32.766" y1="4.826" x2="32.893" y2="4.699" width="0.2" layer="1"/>
+<wire x1="38.481" y1="4.826" x2="33.02" y2="4.826" width="0.2" layer="1"/>
+<wire x1="32.893" y1="4.699" x2="33.02" y2="4.826" width="0.2" layer="1"/>
+<wire x1="38.481" y1="4.826" x2="38.608" y2="4.699" width="0.2" layer="1"/>
+<wire x1="43.815" y1="4.826" x2="38.735" y2="4.826" width="0.2" layer="1"/>
+<wire x1="38.608" y1="4.699" x2="38.735" y2="4.826" width="0.2" layer="1"/>
+<wire x1="43.815" y1="4.826" x2="44.069" y2="4.572" width="0.2" layer="1"/>
 <wire x1="44.069" y1="4.572" x2="44.069" y2="4.699" width="0.2" layer="1"/>
 <wire x1="45.593" y1="6.223" x2="44.069" y2="4.699" width="0.2" layer="1"/>

Commit message: Add files via upload
Parts:
- added J13: (no value), SparkFun-Connectors:1X02_2.54_SCREWTERM
- BTN1, RST: value MOMENTARY-SWITCH-SPST-SMD-5.2-REDUNDANT -> MOMENTARY-SWITCH-SPST-SMD-4.6X2.8MM; device SparkFun-Switches:TACTILE_SWITCH_SMD_5.2MM -> SparkFun-Switches:TACTILE_SWITCH_SMD_4.6X2.8MM
- moved RST 32.0 mm to (43.7, 17.5)
- moved BTN1 0.52 mm to (43.7, 22.2), turned to 0 degrees
Connections:
- net +3V3: now also J13.P2
- net GND: now also J13.P1
Routing:
- net RST: track 40.3 -> 15.0 mm, vias 0 -> 2
- net +3V3: track 72.7 -> 74.9 mm
- net 13: track 18.4 -> 17.3 mm
- net GND: vias 140 -> 144
Other:
- board text added: "-"

Commit message: Add files via upload
Parts:
- removed C11, C12, C13, C14, C15: 100nF, SparkFun-Capacitors:0603
- added R20, R21, R22, R23, R24: 3k, adafruit:R0805
Connections:
- net GND: now also R20.1, R21.1, R22.1, R23.1, R24.1; no longer C11.1, C12.1, C13.1, C14.1, C15.1
- net N$11: now also R23.2; no longer C14.2
- net N$12: now also R24.2; no longer C15.2
- net N$2: now also R20.2; no longer C11.2
- net N$7: now also R21.2; no longer C12.2
- net N$8: now also R22.2; no longer C13.2
