File: v1.1/zb_pt4115_v1.1.sch (EAGLE design)
At the start: 78 parts, among them IC1 68uH, IC2 68uH, IC3 68uH, IC4 68uH, IC5 68uH, IC6 68uH, U1 E72-2G4M05S1F, U2 LM2596T-ADJ/NOPB

Commit message: Add files via upload
Parts:
- added J13: (no value), SparkFun-Connectors:CONN_022.54MM_SCREWTERM
- BTN1, RST: value MOMENTARY-SWITCH-SPST-SMD-5.2-REDUNDANT -> MOMENTARY-SWITCH-SPST-SMD-4.6X2.8MM; device SparkFun-Switches:MOMENTARY-SWITCH-SPST-SMD-5.2-REDUNDANT -> SparkFun-Switches:MOMENTARY-SWITCH-SPST-SMD-4.6X2.8MM
Connections:
- net +3V3: now also J13.2
- net GND: now also J13.1
Changed lines of the file:
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@@
 <part name="MGT3" library="holes" library_urn="urn:adsk.eagle:library:237" deviceset="MOUNT-HOLE" device="3.0" package3d_urn="urn:adsk.eagle:package:14277/1" value="MOUNT-HOLE3.0"/>
 <part name="MGT4" library="holes" library_urn="urn:adsk.eagle:library:237" deviceset="MOUNT-HOLE" device="3.0" package3d_urn="urn:adsk.eagle:package:14277/1"/>
-<part name="RST" library="SparkFun-Switches" library_urn="urn:adsk.eagle:library:535" deviceset="MOMENTARY-SWITCH-SPST" device="-SMD-5.2-REDUNDANT" package3d_urn="urn:adsk.eagle:package:40167/1"/>
+<part name="RST" library="SparkFun-Switches" deviceset="MOMENTARY-SWITCH-SPST" device="-SMD-4.6X2.8MM" package3d_urn="urn:adsk.eagle:package:40176/1"/>
 <part name="GND21" library="supply1" library_urn="urn:adsk.eagle:library:371" deviceset="GND" device=""/>
-<part name="BTN1" library="SparkFun-Switches" library_urn="urn:adsk.eagle:library:535" deviceset="MOMENTARY-SWITCH-SPST" device="-SMD-5.2-REDUNDANT" package3d_urn="urn:adsk.eagle:package:40167/1"/>
+<part name="BTN1" library="SparkFun-Switches" deviceset="MOMENTARY-SWITCH-SPST" device="-SMD-4.6X2.8MM" package3d_urn="urn:adsk.eagle:package:40176/1"/>
 <part name="GND22" library="supply1" library_urn="urn:adsk.eagle:library:371" deviceset="GND" device=""/>
 <part name="C11" library="SparkFun-Capacitors" library_urn="urn:adsk.eagle:library:510" deviceset="2.2NF/2200PF" device="-0603-50V-10%" package3d_urn="urn:adsk.eagle:package:37414/1" value="100nF"/>
@@
 <part name="C20" library="SparkFun-Capacitors" library_urn="urn:adsk.eagle:library:510" deviceset="0.1UF" device="-0603-100V-10%" package3d_urn="urn:adsk.eagle:package:37414/1" value="0.1uF"/>
 <part name="+3V5" library="supply1" library_urn="urn:adsk.eagle:library:371" deviceset="+3V3" device=""/>
+<part name="J13" library="SparkFun-Connectors" library_urn="urn:adsk.eagle:library:513" deviceset="CONN_02" device="2.54MM_SCREWTERM" package3d_urn="urn:adsk.eagle:package:38059/1"/>
+<part name="GND32" library="supply1" library_urn="urn:adsk.eagle:library:371" deviceset="GND" device=""/>
+<part name="+3V6" library="supply1" library_urn="urn:adsk.eagle:library:371" deviceset="+3V3" device=""/>
 </parts>
 <sheets>
@@
 <instance part="+3V5" gate="G$1" x="149.86" y="58.42" smashed="yes">
 <attribute name="VALUE" x="147.32" y="53.34" size="1.778" layer="96" rot="R90"/>
+</instance>
+<instance part="J13" gate="G$1" x="261.62" y="20.32" smashed="yes" rot="R90">
+<attribute name="VALUE" x="266.446" y="17.78" size="1.778" layer="96" font="vector" rot="R90"/>
+<attribute name="NAME" x="256.032" y="17.78" size="1.778" layer="95" font="vector" rot="R90"/>
+</instance>
+<instance part="GND32" gate="1" x="266.7" y="27.94" smashed="yes">
+<attribute name="VALUE" x="264.16" y="25.4" size="1.778" layer="96"/>
+</instance>
+<instance part="+3V6" gate="G$1" x="259.08" y="40.64" smashed="yes">
+<attribute name="VALUE" x="256.54" y="35.56" size="1.778" layer="96" rot="R90"/>
 </instance>
 </instances>
@@
 <wire x1="243.84" y1="35.56" x2="243.84" y2="43.18" width="0.1524" layer="91"/>
 <junction x="243.84" y="35.56"/>
+</segment>
+<segment>
+<pinref part="J13" gate="G$1" pin="1"/>
+<wire x1="261.62" y1="27.94" x2="261.62" y2="33.02" width="0.1524" layer="91"/>
+<wire x1="261.62" y1="33.02" x2="266.7" y2="33.02" width="0.1524" layer="91"/>
+<wire x1="266.7" y1="33.02" x2="266.7" y2="30.48" width="0.1524" layer="91"/>
+<pinref part="GND32" gate="1" pin="GND"/>
 </segment>
 </net>
@@
 <wire x1="236.22" y1="50.8" x2="236.22" y2="48.26" width="0.1524" layer="91"/>
 </segment>
-</net>
+<segment>
+<pinref part="J13" gate="G$1" pin="2"/>
+<pinref part="+3V6" gate="G$1" pin="+3V3"/>
+<wire x1="259.08" y1="27.94" x2="259.08" y2="38.1" width="0.1524" layer="91"/>
+</segment>
+</net>

Commit message: Add files via upload
Parts:
- removed C11, C12, C13, C14, C15: 100nF, SparkFun-Capacitors:2.2NF/2200PF-0603-50V-10%
- added R20, R21, R22, R23, R24: 3k, adafruit:R-US_R0805
Connections:
- net GND: now also R20.1, R21.1, R22.1, R23.1, R24.1; no longer C11.1, C12.1, C13.1, C14.1, C15.1
- net N$11: now also R23.2; no longer C14.2
- net N$12: now also R24.2; no longer C15.2
- net N$2: now also R20.2; no longer C11.2
- net N$7: now also R21.2; no longer C12.2
- net N$8: now also R22.2; no longer C13.2
Changed lines of the file:
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@@
 <part name="BTN1" library="SparkFun-Switches" deviceset="MOMENTARY-SWITCH-SPST" device="-SMD-4.6X2.8MM" package3d_urn="urn:adsk.eagle:package:40176/1"/>
 <part name="GND22" library="supply1" library_urn="urn:adsk.eagle:library:371" deviceset="GND" device=""/>
-<part name="C11" library="SparkFun-Capacitors" library_urn="urn:adsk.eagle:library:510" deviceset="2.2NF/2200PF" device="-0603-50V-10%" package3d_urn="urn:adsk.eagle:package:37414/1" value="100nF"/>
-<part name="C12" library="SparkFun-Capacitors" library_urn="urn:adsk.eagle:library:510" deviceset="2.2NF/2200PF" device="-0603-50V-10%" package3d_urn="urn:adsk.eagle:package:37414/1" value="100nF"/>
-<part name="C13" library="SparkFun-Capacitors" library_urn="urn:adsk.eagle:library:510" deviceset="2.2NF/2200PF" device="-0603-50V-10%" package3d_urn="urn:adsk.eagle:package:37414/1" value="100nF"/>
-<part name="C14" library="SparkFun-Capacitors" library_urn="urn:adsk.eagle:library:510" deviceset="2.2NF/2200PF" device="-0603-50V-10%" package3d_urn="urn:adsk.eagle:package:37414/1" value="100nF"/>
-<part name="C15" library="SparkFun-Capacitors" library_urn="urn:adsk.eagle:library:510" deviceset="2.2NF/2200PF" device="-0603-50V-10%" package3d_urn="urn:adsk.eagle:package:37414/1" value="100nF"/>
+<part name="R20" library="adafruit" library_urn="urn:adsk.eagle:library:420" deviceset="R-US_" device="R0805" package3d_urn="urn:adsk.eagle:package:6240566/1" value="3k"/>
+<part name="R21" library="adafruit" library_urn="urn:adsk.eagle:library:420" deviceset="R-US_" device="R0805" package3d_urn="urn:adsk.eagle:package:6240566/1" value="3k"/>
+<part name="R22" library="adafruit" library_urn="urn:adsk.eagle:library:420" deviceset="R-US_" device="R0805" package3d_urn="urn:adsk.eagle:package:6240566/1" value="3k"/>
+<part name="R23" library="adafruit" library_urn="urn:adsk.eagle:library:420" deviceset="R-US_" device="R0805" package3d_urn="urn:adsk.eagle:package:6240566/1" value="3k"/>
+<part name="R24" library="adafruit" library_urn="urn:adsk.eagle:library:420" deviceset="R-US_" device="R0805" package3d_urn="urn:adsk.eagle:package:6240566/1" value="3k"/>
 <part name="GND18" library="supply1" library_urn="urn:adsk.eagle:library:371" deviceset="GND" device=""/>
 <part name="GND23" library="supply1" library_urn="urn:adsk.eagle:library:371" deviceset="GND" device=""/>
@@
 <attribute name="VALUE" x="15.24" y="33.02" size="1.778" layer="96"/>
 </instance>
-<instance part="C11" gate="G$1" x="170.18" y="93.98" smashed="yes">
-<attribute name="NAME" x="171.704" y="96.901" size="1.778" layer="95" font="vector"/>
-</instance>
-<instance part="C12" gate="G$1" x="226.06" y="93.98" smashed="yes">
-<attribute name="NAME" x="227.584" y="96.901" size="1.778" layer="95" font="vector"/>
-</instance>
-<instance part="C13" gate="G$1" x="284.48" y="93.98" smashed="yes">
-<attribute name="NAME" x="286.004" y="96.901" size="1.778" layer="95" font="vector"/>
-</instance>
-<instance part="C14" gate="G$1" x="340.36" y="93.98" smashed="yes">
-<attribute name="NAME" x="341.884" y="96.901" size="1.778" layer="95" font="vector"/>
-</instance>
-<instance part="C15" gate="G$1" x="401.32" y="93.98" smashed="yes">
-<attribute name="NAME" x="402.844" y="96.901" size="1.778" layer="95" font="vector"/>
-</instance>
-<instance part="GND18" gate="1" x="170.18" y="106.68" smashed="yes" rot="R180">
-<attribute name="VALUE" x="172.72" y="109.22" size="1.778" layer="96" rot="R180"/>
-</instance>
-<instance part="GND23" gate="1" x="226.06" y="104.14" smashed="yes" rot="R180">
-<attribute name="VALUE" x="228.6" y="106.68" size="1.778" layer="96" rot="R180"/>
-</instance>
-<instance part="GND24" gate="1" x="284.48" y="104.14" smashed="yes" rot="R180">
-<attribute name="VALUE" x="287.02" y="106.68" size="1.778" layer="96" rot="R180"/>
-</instance>
-<instance part="GND25" gate="1" x="340.36" y="104.14" smashed="yes" rot="R180">
-<attribute name="VALUE" x="342.9" y="106.68" size="1.778" layer="96" rot="R180"/>
-</instance>
-<instance part="GND26" gate="1" x="401.32" y="104.14" smashed="yes" rot="R180">
-<attribute name="VALUE" x="403.86" y="106.68" size="1.778" layer="96" rot="R180"/>
+<instance part="R20" gate="G$1" x="170.18" y="96.52" smashed="yes" rot="R270">
+<attribute name="NAME" x="173.101" y="97.536" size="1.778" layer="95" font="vector" rot="R270"/>
+</instance>
+<instance part="R21" gate="G$1" x="226.06" y="96.52" smashed="yes" rot="R270">
+<attribute name="NAME" x="228.981" y="94.996" size="1.778" layer="95" font="vector" rot="R270"/>
+</instance>
+<instance part="R22" gate="G$1" x="284.48" y="96.52" smashed="yes" rot="R270">
+<attribute name="NAME" x="287.401" y="94.996" size="1.778" layer="95" font="vector" rot="R270"/>
+</instance>
+<instance part="R23" gate="G$1" x="340.36" y="96.52" smashed="yes" rot="R270">
+<attribute name="NAME" x="343.281" y="94.996" size="1.778" layer="95" font="vector" rot="R270"/>
+</instance>
+<instance part="R24" gate="G$1" x="401.32" y="96.52" smashed="yes" rot="R270">
+<attribute name="NAME" x="404.241" y="94.996" size="1.778" layer="95" font="vector" rot="R270"/>
+</instance>
+<instance part="GND18" gate="1" x="170.18" y="109.22" smashed="yes" rot="R180">
+<attribute name="VALUE" x="172.72" y="111.76" size="1.778" layer="96" rot="R180"/>
+</instance>
+<instance part="GND23" gate="1" x="226.06" y="109.22" smashed="yes" rot="R180">
+<attribute name="VALUE" x="228.6" y="111.76" size="1.778" layer="96" rot="R180"/>
+</instance>
+<instance part="GND24" gate="1" x="284.48" y="109.22" smashed="yes" rot="R180">
+<attribute name="VALUE" x="287.02" y="111.76" size="1.778" layer="96" rot="R180"/>
+</instance>
+<instance part="GND25" gate="1" x="340.36" y="109.22" smashed="yes" rot="R180">
+<attribute name="VALUE" x="342.9" y="111.76" size="1.778" layer="96" rot="R180"/>
+</instance>
+<instance part="GND26" gate="1" x="401.32" y="109.22" smashed="yes" rot="R180">
+<attribute name="VALUE" x="403.86" y="111.76" size="1.778" layer="96" rot="R180"/>
 </instance>
 <instance part="J7" gate="G$1" x="391.16" y="48.26" smashed="yes">
@@
 <segment>
 <pinref part="GND24" gate="1" pin="GND"/>
-<pinref part="C13" gate="G$1" pin="1"/>
-<wire x1="284.48" y1="101.6" x2="284.48" y2="99.06" width="0.1524" layer="91"/>
+<pinref part="R22" gate="G$1" pin="1"/>
+<wire x1="284.48" y1="106.68" x2="284.48" y2="101.6" width="0.1524" layer="91"/>
 </segment>
 <segment>
 <pinref part="GND23" gate="1" pin="GND"/>
-<pinref part="C12" gate="G$1" pin="1"/>
-<wire x1="226.06" y1="101.6" x2="226.06" y2="99.06" width="0.1524" layer="91"/>
+<pinref part="R21" gate="G$1" pin="1"/>
+<wire x1="226.06" y1="106.68" x2="226.06" y2="101.6" width="0.1524" layer="91"/>
 </segment>
 <segment>
 <pinref part="GND25" gate="1" pin="GND"/>
-<pinref part="C14" gate="G$1" pin="1"/>
-<wire x1="340.36" y1="101.6" x2="340.36" y2="99.06" width="0.1524" layer="91"/>
+<pinref part="R23" gate="G$1" pin="1"/>
+<wire x1="340.36" y1="106.68" x2="340.36" y2="101.6" width="0.1524" layer="91"/>
 </segment>
 <segment>
 <pinref part="GND26" gate="1" pin="GND"/>
-<pinref part="C15" gate="G$1" pin="1"/>
-<wire x1="401.32" y1="101.6" x2="401.32" y2="99.06" width="0.1524" layer="91"/>
+<pinref part="R24" gate="G$1" pin="1"/>
+<wire x1="401.32" y1="106.68" x2="401.32" y2="101.6" width="0.1524" layer="91"/>
 </segment>
 <segment>
 <pinref part="GND18" gate="1" pin="GND"/>
-<pinref part="C11" gate="G$1" pin="1"/>
-<wire x1="170.18" y1="104.14" x2="170.18" y2="99.06" width="0.1524" layer="91"/>
+<pinref part="R20" gate="G$1" pin="1"/>
+<wire x1="170.18" y1="106.68" x2="170.18" y2="101.6" width="0.1524" layer="91"/>
 </segment>
 <segment>
@@
 <wire x1="160.02" y1="91.44" x2="165.1" y2="91.44" width="0.1524" layer="91"/>
 <pinref part="R6" gate="G$1" pin="1"/>
-<pinref part="C11" gate="G$1" pin="2"/>
+<pinref part="R20" gate="G$1" pin="2"/>
 <wire x1="165.1" y1="91.44" x2="170.18" y2="91.44" width="0.1524" layer="91"/>
 <junction x="165.1" y="91.44"/>
@@
 <wire x1="215.9" y1="91.44" x2="220.98" y2="91.44" width="0.1524" layer="91"/>
 <pinref part="R7" gate="G$1" pin="1"/>
-<pinref part="C12" gate="G$1" pin="2"/>
+<pinref part="R21" gate="G$1" pin="2"/>
 <wire x1="220.98" y1="91.44" x2="226.06" y2="91.44" width="0.1524" layer="91"/>
 <junction x="220.98" y="91.44"/>
@@
 <wire x1="274.32" y1="91.44" x2="279.4" y2="91.44" width="0.1524" layer="91"/>
 <pinref part="R8" gate="G$1" pin="1"/>
-<pinref part="C13" gate="G$1" pin="2"/>
+<pinref part="R22" gate="G$1" pin="2"/>
 <wire x1="279.4" y1="91.44" x2="284.48" y2="91.44" width="0.1524" layer="91"/>
 <junction x="279.4" y="91.44"/>
@@
 <wire x1="330.2" y1="91.44" x2="335.28" y2="91.44" width="0.1524" layer="91"/>
 <pinref part="R9" gate="G$1" pin="1"/>
-<pinref part="C14" gate="G$1" pin="2"/>
+<pinref part="R23" gate="G$1" pin="2"/>
 <wire x1="335.28" y1="91.44" x2="340.36" y2="91.44" width="0.1524" layer="91"/>
 <junction x="335.28" y="91.44"/>
@@
 <wire x1="391.16" y1="91.44" x2="396.24" y2="91.44" width="0.1524" layer="91"/>
 <pinref part="R10" gate="G$1" pin="1"/>
-<pinref part="C15" gate="G$1" pin="2"/>
+<pinref part="R24" gate="G$1" pin="2"/>
 <wire x1="396.24" y1="91.44" x2="401.32" y2="91.44" width="0.1524" layer="91"/>
 <junction x="396.24" y="91.44"/>
